File: ghost.kicad_pcb (KiCad board)
At the start: 4 copper layers, 43.2 x 52.9 mm, 26 parts, among them J1 MK-12C02

Commit message: Added gerbers
Other:
- board text added: "JLCJLCJLCJLC"
- board text added: "https://github.com/gjlp25/KiCad_Ghosty"
- board text added: "{dblquote}Ghosty{dblquote} by Robert Postma"
